File: board/at2xt.kicad_pcb (KiCad board)
At the start: 2 copper layers, 45.7 x 39.4 mm, 15 parts, among them J1 Conn_01x04, J2 XT, J3 AT, J4 PS/2, U1 MCP1700-3302E_TO92, U2 MSP430G2211IPW14

Commit message: Annotate parts, regenerate PCB, gerbers, and drill file.
Parts:
- C1, C2: value 1u -> 2.2u
- U1: value MCP1700-3302E_TO92 -> MCP1700x-330xxTT

Commit message: Minor silkscreen fixups, swap out regulator for part readily available from Mouser.
Parts:
- U1: footprint Package_TO_SOT_SMD:SOT-23 -> Package_TO_SOT_SMD:SOT-89-3
- moved C4 2.54 mm to (161.3, 64.8)
- moved C1 1.85 mm to (164.5, 60.9)
- moved U1 0.90 mm to (160.0, 59.1)
- moved C2 0.11 mm to (158.8, 55.6)
Connections:
- U1 pad 2: +3.3V -> +5V
- U1 pad 3: +5V -> +3.3V
Routing:
- net +5V: track 59.3 -> 61.0 mm

Commit message: Fix errant value for regulator (wrong identifier, correct package).
Parts:
- U1: value MCP1700x-330xxTT -> MCP1700x-330xxMB
Changed lines of the file:
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@@
       (effects (font (size 1 1) (thickness 0.15)))
     )
-    (fp_text value "MCP1700x-330xxTT" (at 0.3 3.5 90) (layer "F.Fab")
+    (fp_text value "MCP1700x-330xxMB" (at 0.3 3.5 90) (layer "F.Fab")
       (effects (font (size 1 1) (thickness 0.15)))
     )
